File: schematic/PowerSupply.kicad_sch (KiCad schematic)
At the start: 0 parts

Commit message: Create power supply schematic
Parts:
- added C1, C2, C3, C4: 10uF, Capacitor_SMD:C_0603_1608Metric, symbol Device:C
- added D1: LED, LED_SMD:LED_0805_2012Metric, symbol Device:LED
- added J1: 10118194-0011LF, 10118194-0011LF:AMPHENOL_10118194-0011LF, symbol 10118194:10118194-0011LF
- added R1: 740R, Resistor_SMD:R_0603_1608Metric, symbol Device:R
- added TP1: 5V, TestPoint:TestPoint_Pad_D2.0mm, symbol Connector:TestPoint
- added TP2: 3V3, TestPoint:TestPoint_Pad_D2.0mm, symbol Connector:TestPoint
- added TP3: 1V2, TestPoint:TestPoint_Pad_D2.0mm, symbol Connector:TestPoint
- added U1: AMS1117-3.3, Package_TO_SOT_SMD:SOT-223-3_TabPin2, symbol Regulator_Linear:AMS1117-3.3
- added U2: AMS1117-1.2, Package_TO_SOT_SMD:SOT-223-3_TabPin2, symbol Regulator_Linear:AMS1117-1.5
Connections:
- new net: D1.2 (A), R1.2
- new net +1V2: C4.1, TP3.1, U2.2 (VO)
- new net +3V3: C2.1, C3.1, TP2.1, U1.2 (VO), U2.3 (VI)
- new net +5V: C1.1, J1.1 (VBUS), R1.1, TP1.1, U1.3 (VI)
- new net GND: C1.2, C2.2, C3.2, C4.2, D1.1 (K), J1.5 (GND), J1.S1 (SHIELD), J1.S2 (SHIELD), J1.S3 (SHIELD), J1.S4 (SHIELD), J1.S5 (SHIELD), J1.S6 (SHIELD), U1.1 (GND), U2.1 (GND)
- no-connect marks 0 -> 3
Other:
- title: (none) -> iCE40 DevBoard
