File: schematic/PowerSupply.kicad_sch (KiCad schematic)
At the start: 12 parts, among them J1 10118194-0011LF, U1 AMS1117-3.3, U2 AMS1117-1.2

Commit message: Update flash header schematic
Parts:
- J1: footprint 10118194-0011LF:AMPHENOL_10118194-0011LF -> Connector_USB:AMPHENOL_10118194-0011LF
- TP1, TP2, TP3: footprint TestPoint:TestPoint_Pad_D2.0mm -> TestPoint:TestPoint_Pad_D1.0mm
Changed lines of the file:
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@@
       (effects (font (size 1.27 1.27)) (justify left))
     )
-    (property "Footprint" "TestPoint:TestPoint_Pad_D2.0mm" (at 182.88 73.66 0)
+    (property "Footprint" "TestPoint:TestPoint_Pad_D1.0mm" (at 182.88 73.66 0)
       (effects (font (size 1.27 1.27)) hide)
     )
@@
       (effects (font (size 1.27 1.27)))
     )
-    (property "Footprint" "10118194-0011LF:AMPHENOL_10118194-0011LF" (at 68.58 83.82 0)
+    (property "Footprint" "Connector_USB:AMPHENOL_10118194-0011LF" (at 68.58 83.82 0)
       (effects (font (size 1.27 1.27)) (justify bottom) hide)
     )
@@
       (effects (font (size 1.27 1.27)) (justify left))
     )
-    (property "Footprint" "TestPoint:TestPoint_Pad_D2.0mm" (at 246.38 73.66 0)
+    (property "Footprint" "TestPoint:TestPoint_Pad_D1.0mm" (at 246.38 73.66 0)
       (effects (font (size 1.27 1.27)) hide)
     )
@@
       (effects (font (size 1.27 1.27)) (justify left))
     )
-    (property "Footprint" "TestPoint:TestPoint_Pad_D2.0mm" (at 93.98 73.66 0)
-      (effects (font (size 1.27 1.27)) hide)
-    )
+    (property "Footprint" "TestPoint:TestPoint_Pad_D1.0mm" (at 93.98 73.66 0)
+      (effects (font (size 1.27 1.27)) hide)
+    )
